File: x500_pdb.kicad_pcb (KiCad board)
At the start: 2 copper layers, 1 part

Commit message: 4 Layers
Parts:
- removed IC**: QFN50P500X500X80-29N, Library:QFN50P500X500X80-29N
- added C_2V5: 0.1uF, Capacitor_SMD:C_0603_1608Metric_Pad1.08x0.95mm_HandSolder, F.Cu at (110.5, 59.2)
- added C_5V0: 1uF, Capacitor_SMD:C_0603_1608Metric_Pad1.08x0.95mm_HandSolder, F.Cu at (110.5, 61.0)
- added C_BOOT1: 0.1uF, Capacitor_SMD:C_0603_1608Metric_Pad1.08x0.95mm_HandSolder, F.Cu at (110.5, 62.7)
- added C_C1: 3.3nF, Capacitor_SMD:C_0603_1608Metric_Pad1.08x0.95mm_HandSolder, F.Cu at (110.5, 64.5)
- added C_F1: 1uF, Capacitor_SMD:C_0603_1608Metric_Pad1.08x0.95mm_HandSolder, F.Cu at (110.5, 66.2)
- added C_FRQ1: 100pF, Capacitor_SMD:C_0603_1608Metric_Pad1.08x0.95mm_HandSolder, B.Cu at (134.9, 104.0)
- added C_IN1: 47uF, Capacitor_Tantalum_SMD:CP_EIA-7343-20_Kemet-V_HandSolder, F.Cu at (117.1, 104.1)
- added C_IN2: 22uF, Capacitor_SMD:C_1210_3225Metric_Pad1.33x2.70mm_HandSolder, F.Cu at (114.6, 69.7)
- added C_IN3: 0.1uF, Capacitor_SMD:C_1206_3216Metric_Pad1.33x1.80mm_HandSolder, F.Cu at (114.6, 65.8)
- added C_OUT1: 47uF, Capacitor_SMD:C_1206_3216Metric_Pad1.33x1.80mm_HandSolder, F.Cu at (71.7, 94.1)
- added C_OUT2: 47uF, Capacitor_SMD:C_1206_3216Metric_Pad1.33x1.80mm_HandSolder, F.Cu at (71.7, 97.5)
- added F1: Fuse, Fuse:Fuse_1206_3216Metric, F.Cu at (77.5, 94.1)
- added IC1: LM21305SQ_NOPB, LM21305:QFN50P500X500X80-29N, B.Cu at (130.0, 105.0)
- added J1: Conn_01x02, Connector_AMASS:AMASS_XT60PW-M_1x02_P7.20mm_Horizontal, F.Cu at (109.3, 108.6)
- added L1: 3.3uH, Inductor_SMD:L_7.3x7.3_H3.5, F.Cu at (123.6, 92.6)
- added R_C1: 8k2, Resistor_SMD:R_0603_1608Metric_Pad0.98x0.95mm_HandSolder, B.Cu at (124.4, 104.6)
- added R_EN1: 10k, Resistor_SMD:R_0603_1608Metric_Pad0.98x0.95mm_HandSolder, F.Cu at (121.9, 115.5)
- added R_F1: 1R, Capacitor_SMD:C_0201_0603Metric, F.Cu at (110.5, 68.0)
- added R_FB1: 73k2, Resistor_SMD:R_0603_1608Metric_Pad0.98x0.95mm_HandSolder, F.Cu at (121.9, 118.0)
- added R_FB2: 10k, Resistor_SMD:R_0603_1608Metric_Pad0.98x0.95mm_HandSolder, F.Cu at (121.9, 120.5)
- added R_FRQ1: 100k, Resistor_SMD:R_0603_1608Metric_Pad0.98x0.95mm_HandSolder, B.Cu at (140.5, 104.2)
- added R_PG1: 100k, Resistor_SMD:R_0603_1608Metric_Pad0.98x0.95mm_HandSolder, F.Cu at (121.9, 125.5)
Routing:
- net /FREQ: track 0.00 -> 1.59 mm
- added copper zone on In1.Cu, net GND
- added copper zone on In2.Cu, net GND
Other:
- board outline added: 50 x 50 mm
- copper layers 2 -> 4

Commit message: Started routing
Parts:
- added H1: MountingHole, MountingHole:MountingHole_3.2mm_M3, F.Cu at (160.8, 90.2)
- added H2: MountingHole, MountingHole:MountingHole_3.2mm_M3, F.Cu at (160.8, 98.2)
- added H3: MountingHole, MountingHole:MountingHole_3.2mm_M3, F.Cu at (160.8, 106.1)
- added H4: MountingHole, MountingHole:MountingHole_3.2mm_M3, F.Cu at (160.8, 114.1)
- added J2: Conn_01x02, Connector_JST:JST_PH_S2B-PH-K_1x02_P2.00mm_Horizontal, F.Cu at (144.4, 114.0)
- added J3: Conn_01x02, Connector_JST:JST_PH_S2B-PH-K_1x02_P2.00mm_Horizontal, F.Cu at (144.4, 106.0)
- added J4: Conn_01x02, Connector_JST:JST_PH_S2B-PH-K_1x02_P2.00mm_Horizontal, F.Cu at (144.4, 98.1)
- added TP1: TestPoint_Probe, TestPoint:TestPoint_Pad_1.5x1.5mm, F.Cu at (166.6, 88.0)
- added TP2: TestPoint_Probe, TestPoint:TestPoint_Pad_1.5x1.5mm, F.Cu at (166.6, 91.6)
- added TP3: TestPoint_Probe, TestPoint:TestPoint_Pad_1.5x1.5mm, F.Cu at (166.6, 95.1)
- C_2V5, C_5V0, C_BOOT1, C_C1, C_F1, R_FB1, R_FB2, R_PG1: moved to B.Cu
- J1: footprint Connector_AMASS:AMASS_XT60PW-M_1x02_P7.20mm_Horizontal -> easyeda2kicad:CONN-TH_XT60PW-M
- R_EN1: value 10k -> 10K; moved to B.Cu
- R_F1: footprint Capacitor_SMD:C_0201_0603Metric -> Capacitor_SMD:C_0603_1608Metric_Pad1.08x0.95mm_HandSolder; moved to B.Cu
- moved C_2V5 69.7 mm to (135.3, 124.4)
- moved C_5V0 66.5 mm to (135.3, 122.6)
- moved C_BOOT1 63.2 mm to (135.3, 120.9)
- moved C_F1 47.5 mm to (131.4, 108.9), turned to 180 degrees
- moved R_F1 47.3 mm to (131.4, 110.5)
- moved C_C1 40.5 mm to (130.0, 100.0), turned to -90 degrees
- moved F1 39.4 mm to (116.8, 97.9), turned to -90 degrees
- moved C_IN3 38.2 mm to (122.1, 103.3)
- moved C_IN2 37.5 mm to (122.1, 106.4)
- moved R_EN1 10.0 mm to (121.9, 125.5)
- moved R_PG1 10.0 mm to (121.9, 115.5)
- moved R_C1 9.83 mm to (130.0, 96.5), turned to -90 degrees
- moved L1 7.53 mm to (130.1, 96.4)
- moved R_FRQ1 7.08 mm to (134.0, 101.5), turned to 90 degrees
- moved R_FB1 5.02 mm to (121.9, 123.0)
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Connections:
- net /PGOOD_FLAG renamed /PGOOD
- net /VOUT renamed VOUT_5V
- net Net-(IC1-5V0) renamed /5V0
- net Net-(IC1-CBOOT) renamed /CBOOT
- net Net-(IC1-COMP) renamed /COMP
- C_2V5 pad 2: GND -> GNDA
- C_BOOT1 pad 1: Net-(IC1-PVIN_2) -> /SW
- C_F1 pad 1: GND -> /AVIN
- C_F1 pad 2: /AVIN -> GNDA
- C_FRQ1 pad 2: GND -> GNDA
- IC1 pad 10: unconnected-(IC1-PGND_4-Pad10) -> GND
- IC1 pad 14: unconnected-(IC1-AGND_1-Pad14) -> GNDA
- IC1 pad 17: unconnected-(IC1-AGND_2-Pad17) -> GNDA
- IC1 pad 18: unconnected-(IC1-AGND_3-Pad18) -> GNDA
- IC1 pad 19: unconnected-(IC1-AGND_4-Pad19) -> GNDA
- IC1 pad 2: Net-(IC1-PVIN_2) -> BAT+_FUSED
- IC1 pad 20: unconnected-(IC1-AGND_5-Pad20) -> GNDA
- IC1 pad 23: unconnected-(IC1-AVIN_2-Pad23) -> /AVIN
- IC1 pad 24: unconnected-(IC1-AGND_6-Pad24) -> GNDA
- IC1 pad 27: unconnected-(IC1-PVIN_3-Pad27) -> BAT+_FUSED
- IC1 pad 28: unconnected-(IC1-PVIN_4-Pad28) -> BAT+_FUSED
- IC1 pad 3: unconnected-(IC1-SW_1-Pad3) -> /SW
- IC1 pad 4: unconnected-(IC1-SW_2-Pad4) -> /SW
- IC1 pad 5: unconnected-(IC1-SW_3-Pad5) -> /SW
- IC1 pad 6: unconnected-(IC1-SW_4-Pad6) -> /SW
- IC1 pad 7: unconnected-(IC1-PGND_1-Pad7) -> GND
- IC1 pad 8: unconnected-(IC1-PGND_2-Pad8) -> GND
- IC1 pad 9: unconnected-(IC1-PGND_3-Pad9) -> GND
- L1 pad 1: Net-(IC1-PVIN_2) -> /SW
- R_FB2 pad 2: GND -> GNDA
- R_FRQ1 pad 2: GND -> GNDA
Routing:
- net BAT+_FUSED: track 0.00 -> 30.3 mm, vias 0 -> 1
- net +BATT: track 0.00 -> 8.67 mm
- net GND: track 0.00 -> 7.92 mm, vias 0 -> 16
- net /AVIN: track 0.00 -> 3.86 mm
- net Net-(C_C1-Pad1): track 0.00 -> 1.72 mm
- net /COMP: track 0.00 -> 1.69 mm
- net /FREQ: track 1.59 -> 3.23 mm
- net GNDA: track 0.00 -> 1.46 mm
- added copper zone on F.Cu, net VOUT_5V
- added copper zone on In1.Cu, net VOUT_5V
- added copper zone on In2.Cu, net VOUT_5V
- removed copper zone on In1.Cu, net GND
- removed copper zone on In2.Cu, net GND

Commit message: Updating PCB
Parts:
- R_EN1: footprint Resistor_SMD:R_0603_1608Metric_Pad0.98x0.95mm_HandSolder -> Resistor_SMD:R_1206_3216Metric_Pad1.30x1.75mm_HandSolder; moved to F.Cu
- moved C_OUT1 76.3 mm to (147.4, 103.7), turned to -90 degrees
- moved C_OUT2 72.6 mm to (144.1, 103.7), turned to -90 degrees
- moved H3 60.1 mm to (104.0, 125.8)
- moved H1 56.9 mm to (104.2, 84.2)
- moved J2 29.4 mm to (115.8, 120.9), turned to 0 degrees
- moved J4 26.1 mm to (131.8, 120.9), turned to 0 degrees
- moved J3 25.5 mm to (123.8, 120.9), turned to 0 degrees
- moved C_2V5 24.2 mm to (124.8, 102.6), turned to 180 degrees
- moved C_5V0 23.5 mm to (129.7, 99.8), turned to -90 degrees
- moved C_BOOT1 21.5 mm to (131.2, 99.8), turned to -90 degrees
- moved H2 20.3 mm to (146.0, 84.2)
- moved H4 19.3 mm to (145.7, 126.2)
- moved R_EN1 16.0 mm to (122.1, 109.5)
- moved R_C1 14.5 mm to (131.8, 110.9), turned to 0 degrees
- moved R_F1 12.0 mm to (126.5, 99.5)
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Connections:
- R_EN1 pad 1: +BATT -> BAT+_FUSED
- R_F1 pad 1: BAT+_FUSED -> /AVIN
- R_F1 pad 2: /AVIN -> BAT+_FUSED
Routing:
- net VOUT_5V: track 0.00 -> 27.2 mm, vias 0 -> 1
- net /2V5: track 0.00 -> 19.0 mm, vias 0 -> 2
- net BAT+_FUSED: track 30.3 -> 42.9 mm
- net GNDA: track 1.46 -> 11.6 mm
- net /SW: track 0.00 -> 7.03 mm, vias 0 -> 7
- net /EN: track 0.00 -> 5.99 mm, vias 0 -> 1
- net Net-(IC1-FB): track 0.00 -> 5.63 mm
- net /PGOOD: track 0.00 -> 3.15 mm
- net /CBOOT: track 0.00 -> 2.33 mm
- net /5V0: track 0.00 -> 1.93 mm
- net /AVIN: track 3.86 -> 5.25 mm
- net /COMP: track 1.69 -> 2.43 mm
- added copper zone on B.Cu, net /SW
- added copper zone on F.Cu, net /SW
- added copper zone on B.Cu, net BAT+_FUSED
- added copper zone on B.Cu, net GND
- added copper zone on F.Cu, net GND
- added copper zone on In1.Cu, net GND
- added copper zone on B.Cu, net GNDA
- removed copper zone on In1.Cu, net VOUT_5V

Commit message: Cleaning up GND split layer
Parts:
- added NT1: NetTie_2, NetTie:NetTie-2_SMD_Pad2.0mm, B.Cu at (129.5, 92.2)
- TP1, TP2: moved to B.Cu
- moved TP2 39.6 mm to (127.7, 84.1)
- moved TP1 35.3 mm to (131.5, 84.1)
- moved C_5V0 1.52 mm to (131.1, 99.3), turned to 180 degrees
- moved C_BOOT1 1.20 mm to (131.1, 101.0), turned to 180 degrees
Routing:
- net BAT+_FUSED: track 42.9 -> 46.5 mm
- net /5V0: track 1.93 -> 4.74 mm
- net VOUT_5V: track 27.2 -> 25.1 mm
- net /SW: track 7.03 -> 5.03 mm
- net GND: track 7.92 -> 9.29 mm, vias 16 -> 17
- net /CBOOT: track 2.33 -> 1.59 mm
Other:
- board text added: "GND"
- board text added: "GNDA"
